Commit message: Fixed table sliding in Gazebo

File: doc/mesh_filter/urdf/ur5_sensor.urdf.xacro (robot description, xacro)
@@ -11,28 +11,31 @@
     transmission_hw_interface="$(arg transmission_hw_interface)"/>
   <link name="kinect">
+    <visual>
+      <origin rpy="0 0 0" xyz="0 0 0"/>
+      <geometry>
+        <mesh filename="package://moveit_tutorials/doc/mesh_filter/meshes/kinect.dae"/>
+      </geometry>
+    </visual>
     <inertial>
-      <mass value="1e-5"/>
-      <origin xyz="0 0 0" rpy=" 0 0 0"/>
-      <inertia
-          ixx="1e-6" ixy="0" ixz="0"
-          iyy="1e-6" iyz="0"
-          izz="1e-6"
-      />
+      <mass value="0.001"/>
+      <origin xyz="0 0 0"/>
+      <inertia ixx="0.0001" ixy="0.0" ixz="0.0" iyy="0.0001" iyz="0.0" izz="0.0001"/>
     </inertial>
-    <collision name='camera_collision'>
-      <origin xyz="0 0 0" rpy=" 0 0 0"/>
+    <collision>
+      <origin rpy="0 0 0" xyz="0.0 0.0 0.0"/>
       <geometry>
-        <box size=".1 .1 .1"/>
+        <box size="0.07271 0.27794 0.073"/>
       </geometry>
     </collision>
   </link>
-  <joint type="fixed" name="hokuyo_joint">
-    <origin xyz="0.15 -1 0.1" rpy="0 0 0"/>
+  <joint type="fixed" name="kinect_joint">
+    <origin xyz="0.15 -1 0.1" rpy="-1.57 0 0"/>
     <child link="kinect"/>
     <parent link="table"/>
-    <axis xyz="0 1 0" rpy="0 0 0"/>
+    <axis xyz="0 0 0" rpy="0 0 0"/>
     <limit effort="10000" velocity="1000"/>
     <dynamics damping="1.0" friction="1.0"/>
   </joint>
+  <link name="world" />
   <link name="table">
     <visual>
@@ -43,4 +46,12 @@
       <material name="grey"/>
     </visual>
+    <surface>
+      <friction>
+        <ode>
+          <mu>5</mu>
+          <mu2>5</mu2>
+        </ode>
+      </friction>
+    </surface>
     <collision name='camera_collision'>
       <origin rpy="0 0 0" xyz="0 -0.45 -0.03"/>
@@ -50,82 +61,11 @@
     </collision>
   </link>
-  <joint name="table_joint" type="fixed">
+  <joint name="world_table_joint" type="fixed">
+    <parent link="world"/>
+    <child link="table"/>
+  </joint>
+  <joint name="table_arm_joint" type="fixed">
     <parent link="table"/>
     <child link="base_link"/>
   </joint>
-   <joint name="camera_rgb_joint" type="fixed">
-    <origin rpy="0 0 1.57" xyz="0 0 0"/>
-    <parent link="kinect"/>
-    <child link="camera_rgb_frame"/>
-  </joint>
-  <link name="camera_rgb_frame">
-    <inertial>
-      <mass value="0.001"/>
-      <origin xyz="0 0 0"/>
-      <inertia ixx="0.0001" ixy="0.0" ixz="0.0" iyy="0.0001" iyz="0.0" izz="0.0001"/>
-    </inertial>
-  </link>
-  <joint name="camera_rgb_optical_joint" type="fixed">
-    <origin rpy="-1.57079632679 0 -1.57079632679" xyz="0 0 0"/>
-    <parent link="camera_rgb_frame"/>
-    <child link="camera_rgb_optical_frame"/>
-  </joint>
-  <link name="camera_rgb_optical_frame">
-    <inertial>
-      <mass value="0.001"/>
-      <origin xyz="0 0 0"/>
-      <inertia ixx="0.0001" ixy="0.0" ixz="0.0" iyy="0.0001" iyz="0.0" izz="0.0001"/>
-    </inertial>
-  </link>
-  <joint name="camera_joint" type="fixed">
-    <origin rpy="0 0 0" xyz="-0.031 -0.0 -0.016"/>
-    <parent link="camera_rgb_frame"/>
-    <child link="camera_link"/>
-  </joint>
-  <link name="camera_link">
-    <visual>
-      <origin rpy="0 0 1.57079632679" xyz="0 0 0"/>
-      <geometry>
-        <mesh filename="package://picknik_ur5_moveit_config/kinect/meshes/kinect.dae"/>
-      </geometry>
-    </visual>
-    <collision>
-      <origin rpy="0 0 0" xyz="0.0 0.0 0.0"/>
-      <geometry>
-        <box size="0.07271 0.27794 0.073"/>
-      </geometry>
-    </collision>
-    <inertial>
-      <mass value="0.001"/>
-      <origin xyz="0 0 0"/>
-      <inertia ixx="0.0001" ixy="0.0" ixz="0.0" iyy="0.0001" iyz="0.0" izz="0.0001"/>
-    </inertial>
-  </link>
-  <!-- The fixed joints & links below are usually published by static_transformers launched by the OpenNi launch
-     files. However, for Gazebo simulation we need them, so we add them here.
-     (Hence, don't publish them additionally!) -->
-  <joint name="camera_depth_joint" type="fixed">
-    <origin rpy="0 0 0" xyz="0 0.0 0"/>
-    <parent link="camera_rgb_frame"/>
-    <child link="camera_depth_frame"/>
-  </joint>
-  <link name="camera_depth_frame">
-    <inertial>
-      <mass value="0.001"/>
-      <origin xyz="0 0 0"/>
-      <inertia ixx="0.0001" ixy="0.0" ixz="0.0" iyy="0.0001" iyz="0.0" izz="0.0001"/>
-    </inertial>
-  </link>
-  <joint name="camera_depth_optical_joint" type="fixed">
-    <origin rpy="-1.57079632679 0 -1.57079632679" xyz="0 0 0"/>
-    <parent link="camera_depth_frame"/>
-    <child link="camera_depth_optical_frame"/>
-  </joint>
-  <link name="camera_depth_optical_frame">
-    <inertial>
-      <mass value="0.001"/>
-      <origin xyz="0 0 0"/>
-      <inertia ixx="0.0001" ixy="0.0" ixz="0.0" iyy="0.0001" iyz="0.0" izz="0.0001"/>
-    </inertial>
-  </link>
 </robot>

Commit message: Rectified Kinect Orientation

File: doc/mesh_filter/urdf/ur5_sensor.urdf.xacro (robot description, xacro)
@@ -10,31 +10,4 @@
   <xacro:ur5_robot prefix="" joint_limited="false"
     transmission_hw_interface="$(arg transmission_hw_interface)"/>
-  <link name="kinect">
-    <visual>
-      <origin rpy="0 0 0" xyz="0 0 0"/>
-      <geometry>
-        <mesh filename="package://moveit_tutorials/doc/mesh_filter/meshes/kinect.dae"/>
-      </geometry>
-    </visual>
-    <inertial>
-      <mass value="0.001"/>
-      <origin xyz="0 0 0"/>
-      <inertia ixx="0.0001" ixy="0.0" ixz="0.0" iyy="0.0001" iyz="0.0" izz="0.0001"/>
-    </inertial>
-    <collision>
-      <origin rpy="0 0 0" xyz="0.0 0.0 0.0"/>
-      <geometry>
-        <box size="0.07271 0.27794 0.073"/>
-      </geometry>
-    </collision>
-  </link>
-  <joint type="fixed" name="kinect_joint">
-    <origin xyz="0.15 -1 0.1" rpy="-1.57 0 0"/>
-    <child link="kinect"/>
-    <parent link="table"/>
-    <axis xyz="0 0 0" rpy="0 0 0"/>
-    <limit effort="10000" velocity="1000"/>
-    <dynamics damping="1.0" friction="1.0"/>
-  </joint>
   <link name="world" />
   <link name="table">
@@ -65,7 +38,85 @@
     <child link="table"/>
   </joint>
-  <joint name="table_arm_joint" type="fixed">
+  <joint name="table_joint" type="fixed">
     <parent link="table"/>
     <child link="base_link"/>
   </joint>
+  <joint type="fixed" name="table_camera_joint">
+    <origin xyz="0.15 -1 0.1" rpy="0 0 1.57"/>
+    <child link="camera_rgb_frame"/>
+    <parent link="table"/>
+    <axis xyz="0 0 0" rpy="0 0 0"/>
+    <limit effort="10000" velocity="1000"/>
+    <dynamics damping="1.0" friction="1.0"/>
+  </joint>
+  <link name="camera_rgb_frame">
+    <inertial>
+      <mass value="0.001"/>
+      <origin xyz="0 0 0"/>
+      <inertia ixx="0.0001" ixy="0.0" ixz="0.0" iyy="0.0001" iyz="0.0" izz="0.0001"/>
+    </inertial>
+  </link>
+  <joint name="camera_rgb_optical_joint" type="fixed">
+    <origin rpy="-1.57079632679 0 -1.57079632679" xyz="0 0 0"/>
+    <parent link="camera_rgb_frame"/>
+    <child link="camera_rgb_optical_frame"/>
+  </joint>
+  <link name="camera_rgb_optical_frame">
+    <inertial>
+      <mass value="0.001"/>
+      <origin xyz="0 0 0"/>
+      <inertia ixx="0.0001" ixy="0.0" ixz="0.0" iyy="0.0001" iyz="0.0" izz="0.0001"/>
+    </inertial>
+  </link>
+  <joint name="camera_joint" type="fixed">
+    <origin rpy="0 0 0" xyz="-0.031 -0.0 -0.016"/>
+    <parent link="camera_rgb_frame"/>
+    <child link="camera_link"/>
+  </joint>
+  <link name="camera_link">
+    <visual>
+      <origin rpy="0 0 0" xyz="0 0 0"/>
+      <geometry>
+        <mesh filename="package://moveit_tutorials/doc/mesh_filter/meshes/kinect.dae"/>
+      </geometry>
+    </visual>
+    <collision>
+      <origin rpy="0 0 0" xyz="0.0 0.0 0.0"/>
+      <geometry>
+        <box size="0.07271 0.27794 0.073"/>
+      </geometry>
+    </collision>
+    <inertial>
+      <mass value="0.001"/>
+      <origin xyz="0 0 0"/>
+      <inertia ixx="0.0001" ixy="0.0" ixz="0.0" iyy="0.0001" iyz="0.0" izz="0.0001"/>
+    </inertial>
+  </link>
+  <!-- The fixed joints & links below are usually published by static_transformers launched by the OpenNi launch
+     files. However, for Gazebo simulation we need them, so we add them here.
+     (Hence, don't publish them additionally!) -->
+  <joint name="camera_depth_joint" type="fixed">
+    <origin rpy="0 0 0" xyz="0 0.0 0"/>
+    <parent link="camera_rgb_frame"/>
+    <child link="camera_depth_frame"/>
+  </joint>
+  <link name="camera_depth_frame">
+    <inertial>
+      <mass value="0.001"/>
+      <origin xyz="0 0 0"/>
+      <inertia ixx="0.0001" ixy="0.0" ixz="0.0" iyy="0.0001" iyz="0.0" izz="0.0001"/>
+    </inertial>
+  </link>
+  <joint name="camera_depth_optical_joint" type="fixed">
+    <origin rpy="-1.57079632679 0 -1.57079632679" xyz="0 0 0"/>
+    <parent link="camera_depth_frame"/>
+    <child link="camera_depth_optical_frame"/>
+  </joint>
+  <link name="camera_depth_optical_frame">
+    <inertial>
+      <mass value="0.001"/>
+      <origin xyz="0 0 0"/>
+      <inertia ixx="0.0001" ixy="0.0" ixz="0.0" iyy="0.0001" iyz="0.0" izz="0.0001"/>
+    </inertial>
+  </link>
 </robot>

Commit message: Changes to documentation (as suggested by Dave)

File: doc/mesh_filter/urdf/ur5_sensor.urdf.xacro (robot description, xacro)
@@ -79,7 +79,7 @@
     <visual>
       <origin rpy="0 0 0" xyz="0 0 0"/>
-      <geometry>
+      <!-- <geometry>
         <mesh filename="package://moveit_tutorials/doc/mesh_filter/meshes/kinect.dae"/>
-      </geometry>
+      </geometry> -->
     </visual>
     <collision>

Commit message: Add tutorial to index.rst

File: doc/mesh_filter/urdf/ur5_sensor.urdf.xacro (robot description, xacro)
@@ -79,7 +79,7 @@
     <visual>
       <origin rpy="0 0 0" xyz="0 0 0"/>
-      <!-- <geometry>
+      <geometry>
         <mesh filename="package://moveit_tutorials/doc/mesh_filter/meshes/kinect.dae"/>
-      </geometry> -->
+      </geometry>
     </visual>
     <collision>

Commit message: Fix for install workspace

File: doc/mesh_filter/urdf/ur5_sensor.urdf.xacro (robot description, xacro)
@@ -3,7 +3,46 @@
        name="ur5" >
   <xacro:arg name="transmission_hw_interface" default="hardware_interface/PositionJointInterface"/>
+  <xacro:arg name="cameraMesh" default=""/>
   <!-- common stuff -->
   <xacro:include filename="$(find ur_description)/urdf/common.gazebo.xacro" />
-  <include filename="$(find moveit_tutorials)/doc/mesh_filter/urdf/ur5_sensor.gazebo" />
+  <!-- Add sensor -->
+  <robot>
+  <gazebo reference="camera_depth_frame">
+    <sensor name="kinect_camera" type="depth">
+      <update_rate>20</update_rate>
+      <camera>
+        <horizontal_fov>1.047198</horizontal_fov>
+        <image>
+          <width>640</width>
+          <height>480</height>
+          <format>B8G8R8</format>
+        </image>
+        <clip>
+          <near>0.05</near>
+          <far>3</far>
+        </clip>
+      </camera>
+      <plugin name="kinect_controller" filename="libgazebo_ros_openni_kinect.so">
+        <baseline>0.1</baseline>
+        <alwaysOn>true</alwaysOn>
+        <updateRate>10</updateRate>
+        <cameraName>camera_ir</cameraName>
+        <imageTopicName>/camera/color/image_raw</imageTopicName>
+        <cameraInfoTopicName>/camera/color/camera_info</cameraInfoTopicName>
+        <depthImageTopicName>/camera/depth/image_raw</depthImageTopicName>
+        <depthImageCameraInfoTopicName>/camera/depth/camera_info</depthImageCameraInfoTopicName>
+        <pointCloudTopicName>/camera/depth/points</pointCloudTopicName>
+        <frameName>camera_depth_optical_frame</frameName>
+        <distortion_k1>0.0</distortion_k1>
+        <distortion_k2>0.0</distortion_k2>
+        <distortion_k3>0.0</distortion_k3>
+        <distortion_t1>0.0</distortion_t1>
+        <distortion_t2>0.0</distortion_t2>
+        <pointCloudCutoff>0.16</pointCloudCutoff>
+        <pointCloudCutoffMax>10.0</pointCloudCutoffMax>
+      </plugin>
+    </sensor>
+  </gazebo>
+  </robot>
   <!-- ur5 -->
   <xacro:include filename="$(find ur_description)/urdf/ur5.urdf.xacro" />
@@ -80,5 +119,5 @@
       <origin rpy="0 0 0" xyz="0 0 0"/>
       <geometry>
-        <mesh filename="package://moveit_tutorials/doc/mesh_filter/meshes/kinect.dae"/>
+        <mesh filename="file://$(arg cameraMesh)"/>
       </geometry>
     </visual>

Commit message: Add dependencies to package.xml

File: doc/mesh_filter/urdf/ur5_sensor.urdf.xacro (robot description, xacro)
@@ -3,46 +3,9 @@
        name="ur5" >
   <xacro:arg name="transmission_hw_interface" default="hardware_interface/PositionJointInterface"/>
-  <xacro:arg name="cameraMesh" default=""/>
+  <xacro:arg name="resource_dir" default=""/>
   <!-- common stuff -->
   <xacro:include filename="$(find ur_description)/urdf/common.gazebo.xacro" />
   <!-- Add sensor -->
-  <robot>
-  <gazebo reference="camera_depth_frame">
-    <sensor name="kinect_camera" type="depth">
-      <update_rate>20</update_rate>
-      <camera>
-        <horizontal_fov>1.047198</horizontal_fov>
-        <image>
-          <width>640</width>
-          <height>480</height>
-          <format>B8G8R8</format>
-        </image>
-        <clip>
-          <near>0.05</near>
-          <far>3</far>
-        </clip>
-      </camera>
-      <plugin name="kinect_controller" filename="libgazebo_ros_openni_kinect.so">
-        <baseline>0.1</baseline>
-        <alwaysOn>true</alwaysOn>
-        <updateRate>10</updateRate>
-        <cameraName>camera_ir</cameraName>
-        <imageTopicName>/camera/color/image_raw</imageTopicName>
-        <cameraInfoTopicName>/camera/color/camera_info</cameraInfoTopicName>
-        <depthImageTopicName>/camera/depth/image_raw</depthImageTopicName>
-        <depthImageCameraInfoTopicName>/camera/depth/camera_info</depthImageCameraInfoTopicName>
-        <pointCloudTopicName>/camera/depth/points</pointCloudTopicName>
-        <frameName>camera_depth_optical_frame</frameName>
-        <distortion_k1>0.0</distortion_k1>
-        <distortion_k2>0.0</distortion_k2>
-        <distortion_k3>0.0</distortion_k3>
-        <distortion_t1>0.0</distortion_t1>
-        <distortion_t2>0.0</distortion_t2>
-        <pointCloudCutoff>0.16</pointCloudCutoff>
-        <pointCloudCutoffMax>10.0</pointCloudCutoffMax>
-      </plugin>
-    </sensor>
-  </gazebo>
-  </robot>
+  <xacro:include filename="$(arg resource_dir)/urdf/ur5_sensor.gazebo" />
   <!-- ur5 -->
   <xacro:include filename="$(find ur_description)/urdf/ur5.urdf.xacro" />
@@ -119,5 +82,5 @@
       <origin rpy="0 0 0" xyz="0 0 0"/>
       <geometry>
-        <mesh filename="file://$(arg cameraMesh)"/>
+        <mesh filename="file://$(arg resource_dir)/meshes/kinect.dae"/>
       </geometry>
     </visual>

Commit message: Change layout in install space

File: doc/mesh_filter/urdf/ur5_sensor.urdf.xacro (robot description, xacro)
@@ -7,5 +7,5 @@
   <xacro:include filename="$(find ur_description)/urdf/common.gazebo.xacro" />
   <!-- Add sensor -->
-  <xacro:include filename="$(arg resource_dir)/urdf/kinect_camera.gazebo" />
+  <include filename="$(find moveit_tutorials)/doc/mesh_filter/urdf/kinect_camera.gazebo" />
   <!-- ur5 -->
   <xacro:include filename="$(find ur_description)/urdf/ur5.urdf.xacro" />
@@ -82,5 +82,5 @@
       <origin rpy="0 0 0" xyz="0 0 0"/>
       <geometry>
-        <mesh filename="file://$(arg resource_dir)/meshes/kinect.dae"/>
+        <mesh filename="package://moveit_tutorials/doc/mesh_filter/meshes/kinect.dae"/>
       </geometry>
     </visual>

Commit message: relatively stable

File: doc/mesh_filter/urdf/ur5_sensor.urdf.xacro (robot description, xacro)
@@ -1,53 +1,20 @@
 <?xml version="1.0"?>
-<robot xmlns:xacro="http://wiki.ros.org/xacro"
-       name="ur5" >
-  <xacro:arg name="transmission_hw_interface" default="hardware_interface/PositionJointInterface"/>
-  <xacro:arg name="resource_dir" default=""/>
-  <!-- common stuff -->
-  <xacro:include filename="$(find ur_description)/urdf/common.gazebo.xacro" />
-  <!-- Add sensor -->
-  <include filename="$(find moveit_tutorials)/doc/mesh_filter/urdf/kinect_camera.gazebo" />
-  <!-- ur5 -->
-  <xacro:include filename="$(find ur_description)/urdf/ur5.urdf.xacro" />
-  <xacro:ur5_robot prefix="" joint_limited="false"
-    transmission_hw_interface="$(arg transmission_hw_interface)"/>
-  <link name="world" />
-  <link name="table">
-    <visual>
-      <origin rpy="0 0 0" xyz="0 -0.45 -0.03"/>
-      <geometry>
-        <box size="0.6 1.2 0.05"/>
-      </geometry>
-      <material name="grey"/>
-    </visual>
-    <surface>
-      <friction>
-        <ode>
-          <mu>5</mu>
-          <mu2>5</mu2>
-        </ode>
-      </friction>
-    </surface>
-    <collision name='camera_collision'>
-      <origin rpy="0 0 0" xyz="0 -0.45 -0.03"/>
-      <geometry>
-        <box size="0.6 1.2 0.05"/>
-      </geometry>
-    </collision>
-  </link>
-  <joint name="world_table_joint" type="fixed">
-    <parent link="world"/>
-    <child link="table"/>
-  </joint>
-  <!-- Attach UR5 to table -->
-  <joint name="table_joint" type="fixed">
-    <parent link="table"/>
-    <child link="base_link"/>
-  </joint>
-  <!-- Attach Kinect to table -->
-  <joint type="fixed" name="table_camera_joint">
+<robot xmlns:xacro="http://www.ros.org/wiki/xacro" name="ur5_world">
+  <!-- Include UR5 -->
+  <xacro:arg name="joint_limit_params" default="$(find ur_description)/config/ur5/joint_limits.yaml"/>
+  <xacro:arg name="kinematics_params" default="$(find ur_description)/config/ur5/default_kinematics.yaml"/>
+  <xacro:arg name="physical_params" default="$(find ur_description)/config/ur5/physical_parameters.yaml"/>
+  <xacro:arg name="visual_params" default="$(find ur_description)/config/ur5/visual_parameters.yaml"/>
+  <xacro:arg name="robot_model" default="ur5"/>
+  <xacro:include filename="$(find ur_gazebo)/urdf/ur.xacro"/>
+  <!-- Define the grey material -->
+  <material name="grey">
+    <color rgba="0.5 0.5 0.5 1.0"/>
+  </material>
+<!-- Attach Kinect to world -->
+  <joint type="fixed" name="world_camera_joint">
     <origin xyz="0.15 -1 0.1" rpy="0 0 1.57"/>
     <child link="camera_rgb_frame"/>
-    <parent link="table"/>
+    <parent link="world"/>
     <axis xyz="0 0 0" rpy="0 0 0"/>
     <limit effort="10000" velocity="1000"/>
@@ -124,3 +91,53 @@
     </inertial>
   </link>
+  <!-- GAZEBO PLUGIN -->
+  <!-- Left/Depth camera -->
+  <gazebo reference="camera_link">
+    <material> Gazebo/DarkGrey </material>
+  </gazebo>
+  <gazebo reference="camera_depth_frame">
+    <sensor type="depth" name="kinect_camera">
+      <always_on>true</always_on>
+      <update_rate>15.0</update_rate>
+      <visualize>false</visualize>
+      <camera name="kinect_camera">
+        <horizontal_fov>1.7633</horizontal_fov>
+        <image>
+          <height>720</height>
+          <width>1280</width>
+          <format>R8G8B8</format>
+        </image>
+        <clip>
+          <near>0.1</near>
+          <far>300</far>
+        </clip>
+        <noise>
+          <type>gaussian</type>
+          <mean>0.0</mean>
+          <stddev>0.007</stddev>
+        </noise>
+      </camera>
+      <plugin name="camera_controller" filename="libgazebo_ros_openni_kinect.so">
+        <cameraName>camera_ir</cameraName>
+        <imageTopicName>left/image_rect_color</imageTopicName>
+        <imageTopicName>/camera/color/image_raw</imageTopicName>
+        <cameraInfoTopicName>/camera/color/camera_info</cameraInfoTopicName>
+        <depthImageTopicName>/camera/depth/image_raw</depthImageTopicName>
+        <depthImageCameraInfoTopicName>/camera/depth/camera_info</depthImageCameraInfoTopicName>
+        <pointCloudTopicName>/camera/depth/points</pointCloudTopicName>
+        <frameName>camera_depth_optical_frame</frameName>
+        <pointCloudCutoff>0.1</pointCloudCutoff>
+        <distortionK1>0</distortionK1>
+        <distortionK2>0</distortionK2>
+        <distortionK3>0</distortionK3>
+        <distortionT1>0</distortionT1>
+        <distortionT2>0</distortionT2>
+        <CxPrime>0</CxPrime>
+        <Cx>0</Cx>
+        <Cy>0</Cy>
+        <focalLength>0</focalLength>
+        <hackBaseline>0</hackBaseline>
+      </plugin>
+    </sensor>
+  </gazebo>
 </robot>
